Commit message: Config all file

File: nbt_bot/description/lidar.xacro (robot description, xacro)
@@ -1,20 +1,20 @@
 <?xml version="1.0"?>
-<robot xmlns:xacro="http://www.ros.org/wiki/xacro" >
+<robot xmlns:xacro="http://www.ros.org/wiki/xacro"  name="robot">
     <joint name="laser_joint" type="fixed">
         <parent link="chassis"/>
-        <child link="laser_frame"/>
-        <origin xyz="0.15 0 0.20" rpy="0 0 3.14159"/>
+        <child link="laser"/>
+        <origin xyz="0.22 0 0.15" rpy="0 0 ${pi}"/>
     </joint>
-    <link name="laser_frame">
+    <link name="laser">
         <visual>
             <geometry>
-                <cylinder radius="0.05" length="0.04"/>
+                <cylinder radius="0.025" length="0.02"/>
             </geometry>
             <material name="black"/>
         </visual>
         <visual>
-            <origin xyz="0 0 -0.05"/>
+            <origin xyz="0 0 -0.02"/>
             <geometry>
-                <cylinder radius="0.01" length="0.1"/>
+                <box size="0.05 0.05 0.02"/>
             </geometry>
             <material name="black"/>
@@ -22,21 +22,22 @@
         <collision>
             <geometry>
-                <cylinder radius="0.05" length="0.04"/>
+                <cylinder radius="0.025" length="0.02"/>
             </geometry>
         </collision>
-        <xacro:inertial_cylinder mass="0.1" length="0.04" radius="0.05">
+        <xacro:inertial_cylinder mass="0.1" length="0.02" radius="0.025">
             <origin xyz="0 0 0" rpy="0 0 0"/>
         </xacro:inertial_cylinder>
     </link>
     <gazebo reference="laser_frame">
-        <material>Gazebo/Black</material>
+        <material>Gazebo/Red</material>
         <sensor name="laser" type="ray">
-            <pose> 0 0 0 0 0 0 </pose>
-            <visualize>true</visualize>
+            <pose> 0 0 0 0</pose>
+            <visualize>false</visualize>
             <update_rate>10</update_rate>
             <ray>
                 <scan>
                     <horizontal>
-                        <samples>360</samples>
+                        <sample>360</sample>
+                        <resolution>1</resolution>
                         <min_angle>-3.14</min_angle>
                         <max_angle>3.14</max_angle>
@@ -45,5 +46,6 @@
                 <range>
                     <min>0.3</min>
-                    <max>12</max>
+                    <max>5</max>
+                    <resolution>0.01</resolution>
                 </range>
             </ray>

File: nbt_bot/description/robot_core.xacro (robot description, xacro)
@@ -1,27 +1,7 @@
 <?xml version="1.0"?>
-<robot xmlns:xacro="http://www.ros.org/wiki/xacro" >
+<robot xmlns:xacro="http://www.ros.org/wiki/xacro">
     <xacro:include filename="inertial_macros.xacro"/>
-    <xacro:property name="chassis_length" value="0.30"/>
-    <xacro:property name="chassis_width" value="0.16"/>
-    <xacro:property name="chassis_height" value="0.11"/>
-    <xacro:property name="chassis_mass" value="1.0"/>
-    <xacro:property name="wheel_radius" value="0.033"/>
-    <xacro:property name="wheel_thickness" value="0.026"/>
-    <xacro:property name="wheel_mass" value="0.05"/>
-    <xacro:property name="wheel_offset_x" value="0.10"/>
-    <xacro:property name="wheel_offset_y" value="0.10"/>
-    <xacro:property name="wheel_offset_z" value="0.01"/>
-    <xacro:property name="caster_wheel_radius_left" value="0.033"/>
-    <xacro:property name="caster_wheel_mass_left" value="0.01"/>
-    <xacro:property name="caster_wheel_offset_x_left" value="0.27"/>
-    <xacro:property name="caster_wheel_offset_y_left" value="0.05"/>
-    <xacro:property name="caster_wheel_offset_z_left" value="0.01"/>
-    <xacro:property name="caster_wheel_radius_right" value="0.033"/>
-    <xacro:property name="caster_wheel_mass_right" value="0.01"/>
-    <xacro:property name="caster_wheel_offset_x_right" value="0.27"/>
-    <xacro:property name="caster_wheel_offset_y_right" value="-0.05"/>
-    <xacro:property name="caster_wheel_offset_z_right" value="0.01"/>
     <material name="white">
-        <color rgba="1 1 1 1" />
+        <color rgba="1 1 1 1"/>
     </material>
     <material name="orange">
@@ -31,14 +11,14 @@
         <color rgba="0.2 0.2 1 1"/>
     </material>
+    <material name="red">
+        <color rgba="1 0 0 1"/>
+    </material>
     <material name="black">
         <color rgba="0 0 0 1"/>
-    </material>
-    <material name="red">
-        <color rgba="1 0 0 1"/>
     </material>
     <!-- BASE LINK -->
     <link name="base_link">
     </link>
-    <!-- BASE_FOOTPRINT LINK -->
+    <!-- BASE_FOOTPRINT_LINK -->
     <joint name="base_footprint_joint" type="fixed">
         <parent link="base_link"/>
@@ -52,22 +32,22 @@
         <parent link="base_link"/>
         <child link="chassis"/>
-        <origin xyz="${-wheel_offset_x} 0 ${-wheel_offset_z}"/>
+        <origin xyz="-0.1 0 0"/>
     </joint>
     <link name="chassis">
         <visual>
-            <origin xyz="${chassis_length/2} 0 ${chassis_height/2}"/>
+            <origin xyz="0.17 0 0.0925"/>
             <geometry>
-                <box size="${chassis_length} ${chassis_width} ${chassis_height}"/>
+                <box size="0.2 0.17 0.055"/>
             </geometry>
-            <material name="orange"/>
+            <material name="white"/>
         </visual>
         <collision>
-            <origin xyz="${chassis_length/2} 0 ${chassis_height/2}"/>
+            <origin xyz="0.17 0 0.0925"/>
             <geometry>
-                <box size="${chassis_length} ${chassis_width} ${chassis_height}"/>
+                <box size="0.2 0.17 0.055"/>
             </geometry>
         </collision>
-        <xacro:inertial_box mass="0.5" x="${chassis_length}" y="${chassis_width}" z="${chassis_height}">
-            <origin xyz="${chassis_length/2} 0 ${chassis_height/2}" rpy="0 0 0"/>
+        <xacro:inertial_box mass="0.5" x="0.2" y="0.17" z="0.1">
+            <origin xyz="0.17 0 0.0925" rpy="0 0 0"/>
         </xacro:inertial_box>
     </link>
@@ -79,5 +59,5 @@
         <parent link="base_link"/>
         <child link="left_wheel"/>
-        <origin xyz="0 ${wheel_offset_y} 0" rpy="-${pi/2} 0 0" />
+        <origin xyz="0.0175 0.1 0.0325" rpy="-${pi/2} 0 0"/>
         <axis xyz="0 0 1"/>
     </joint>
@@ -85,5 +65,5 @@
         <visual>
             <geometry>
-                <cylinder radius="${wheel_radius}" length="${wheel_thickness}"/>
+                <cylinder radius="0.0325" length="0.027"/>
             </geometry>
             <material name="blue"/>
@@ -91,8 +71,8 @@
         <collision>
             <geometry>
-                <sphere radius="${wheel_radius}"/>
+                <cylinder radius="0.0325" length="0.027"/>
             </geometry>
         </collision>
-        <xacro:inertial_cylinder mass="${wheel_mass}" length="${wheel_thickness}" radius="${wheel_radius}">
+        <xacro:inertial_cylinder mass="0.1" length="0.027" radius="0.0325">
             <origin xyz="0 0 0" rpy="0 0 0"/>
         </xacro:inertial_cylinder>
@@ -105,5 +85,5 @@
         <parent link="base_link"/>
         <child link="right_wheel"/>
-        <origin xyz="0 ${-wheel_offset_y} 0" rpy="${pi/2} 0 0" />
+        <origin xyz="0.0175 -0.1 0.0325" rpy="${pi/2} 0 0"/>
         <axis xyz="0 0 -1"/>
     </joint>
@@ -111,5 +91,5 @@
         <visual>
             <geometry>
-                <cylinder radius="${wheel_radius}" length="${wheel_thickness}"/>
+                <cylinder radius="0.0325" length="0.027"/>
             </geometry>
             <material name="blue"/>
@@ -117,8 +97,8 @@
         <collision>
             <geometry>
-                <sphere radius="${wheel_radius}"/>
+                <cylinder radius="0.0325" length="0.027"/>
             </geometry>
         </collision>
-        <xacro:inertial_cylinder mass="${wheel_mass}" length="${wheel_thickness}" radius="${wheel_radius}">
+        <xacro:inertial_cylinder mass="0.1" length="0.027" radius="0.0325">
             <origin xyz="0 0 0" rpy="0 0 0"/>
         </xacro:inertial_cylinder>
@@ -127,15 +107,14 @@
         <material>Gazebo/Blue</material>
     </gazebo>
-    <!-- CASTER WHEEL LEFT LINK -->
-    <joint name="caster_wheel_joint_left" type="fixed">
+    <!-- CASTER WHEEL LINK -->
+    <joint name="caster_wheel_joint" type="fixed">
         <parent link="chassis"/>
-        <child link="caster_wheel_left"/>
-        <origin xyz="${caster_wheel_offset_x_left} ${caster_wheel_offset_y_left}
-        ${caster_wheel_offset_z_left}"/>
+        <child link="caster_wheel"/>
+        <origin xyz="0.225 0 0.0325"/>
     </joint>
-    <link name="caster_wheel_left">
+    <link name="caster_wheel">
         <visual>
             <geometry>
-                <sphere radius="${caster_wheel_radius_left}"/>
+                <sphere radius="0.0325"/>
             </geometry>
             <material name="white"/>
@@ -143,62 +122,29 @@
         <collision>
             <geometry>
-                <sphere radius="${caster_wheel_radius_left}"/>
+                <sphere radius="0.0325"/>
             </geometry>
         </collision>
-        <xacro:inertial_sphere mass="${caster_wheel_mass_left}" radius="${caster_wheel_radius_left}">
+        <xacro:inertial_sphere mass="0.1" radius="0.0325">
             <origin xyz="0 0 0" rpy="0 0 0"/>
         </xacro:inertial_sphere>
     </link>
-    <gazebo reference="caster_wheel_left">
-        <material>Gazebo/White</material>
+    <gazebo reference="caster_wheel">
+        <material>Gazebo/Black</material>
         <mu1 value="0.001"/>
         <mu2 value="0.001"/>
     </gazebo>
-<!-- CASTER WHEEL RIGHT LINK -->
-    <joint name="caster_wheel_joint_right" type="fixed">
-        <parent link="chassis"/>
-        <child link="caster_wheel_right"/>
-        <origin xyz="${caster_wheel_offset_x_right} ${caster_wheel_offset_y_right}
-        ${caster_wheel_offset_z_right}"/>
+    <!-- เพิ่ม IMU link ใน URDF -->
+    <link name="imu_link">
+    <visual>
+        <geometry>
+        <box size="0.02 0.02 0.01"/>
+        </geometry>
+        <material name="red"/>
+    </visual>
+    </link>
+    <joint name="imu_joint" type="fixed">
+    <parent link="chassis"/>
+    <child link="imu_link"/>
+    <origin xyz="0.15 0 0.095" rpy="0 0 0"/>
     </joint>
-    <link name="caster_wheel_right">
-        <visual>
-            <geometry>
-                <sphere radius="${caster_wheel_radius_right}"/>
-            </geometry>
-            <material name="white"/>
-        </visual>
-        <collision>
-            <geometry>
-                <sphere radius="${caster_wheel_radius_right}"/>
-            </geometry>
-        </collision>
-        <xacro:inertial_sphere mass="${caster_wheel_mass_right}" radius="${caster_wheel_radius_right}">
-            <origin xyz="0 0 0" rpy="0 0 0"/>
-        </xacro:inertial_sphere>
-    </link>
-    <gazebo reference="caster_wheel_right">
-        <material>Gazebo/White</material>
-        <mu1 value="0.001"/>
-        <mu2 value="0.001"/>
-    </gazebo>
-    <!-- imu -->
-    <joint name="imu_joint" type="fixed">
-        <parent link="chassis"/>
-        <child link="imu_link"/>
-        <origin xyz="0.15 0 0.055" rpy="0 0 0"/>
-    </joint>
-    <link name="imu_link">
-        <visual>
-            <geometry>
-                <box size="0.05 0.05 0.05"/>
-            </geometry>
-            <material name="red"/>
-        </visual>
-        <collision>
-            <geometry>
-                <box size="0.05 0.05 0.05"/>
-            </geometry>
-        </collision>
-    </link>
 </robot>

File: nbt_bot/description/ros2_control.xacro (robot description, xacro)
@@ -8,13 +8,13 @@
                 <param name="right_wheel_name">right_wheel_joint</param>
                 <param name="loop_rate">30</param>
-                <param name="device">/dev/ttyACM0</param>
+                <param name="device">/dev/arduino_nano</param>
                 <param name="baud_rate">57600</param>
                 <param name="timeout">1000</param>
-                <param name="enc_counts_per_rev">2250</param>
+                <param name="enc_counts_per_rev">616</param>
             </hardware>
             <joint name="left_wheel_joint">
                 <command_interface name="velocity">
-                    <param name="min">-10</param>
-                    <param name="max">10</param>
+                    <param name="min">-0.2</param>
+                    <param name="max">0.2</param>
                 </command_interface>
                 <state_interface name="velocity"/>
@@ -23,6 +23,6 @@
             <joint name="right_wheel_joint">
                 <command_interface name="velocity">
-                    <param name="min">-10</param>
-                    <param name="max">10</param>
+                    <param name="min">-0.2</param>
+                    <param name="max">0.2</param>
                 </command_interface>
                 <state_interface name="velocity"/>
@@ -30,5 +30,5 @@
             </joint>
         </ros2_control>
-        <ros2_control name='MPU6050' type='sensor'>
+        <!-- <ros2_control name='MPU6050' type='sensor'>
             <hardware>
                 <plugin>mpu6050_imu_broadcaster/MPU6050Hardware</plugin>
@@ -48,5 +48,5 @@
                 <state_interface name='linear_acceleration.z'/>
             </sensor>
-        </ros2_control>
+        </ros2_control>         -->
     </xacro:unless>
     <xacro:if value="$(arg sim_mode)">
